File: Test LED Matrix/Test LED Matrix.kicad_sch (KiCad schematic)
At the start: 0 parts

Commit message: cbcbc
Parts:
- added D1, D10, D11, D12, D13, D14, D15, D16, D17, D18, D19, D2, D20, D21, D22, D23, D24, D25, D26, D27, D28, D29, D3, D30, D31, D32, D33, D34, D35, D36, D37, D38, D39, D4, D40, D41, D42, D43, D44, D45, D46, D47, D48, D49, D5, D50, D51, D52, D53, D54, D55, D56, D57, D58, D59, D6, D60, D61, D62, D63, D64, D7, D8, D9: WS2812B, LED_SMD:LED_WS2812B_PLCC4_5.0x5.0mm_P3.2mm, symbol LED:WS2812B
- added J1: Conn_01x04_Pin, Connector_PinSocket_2.54mm:PinSocket_1x04_P2.54mm_Vertical, symbol Connector:Conn_01x04_Pin
- added R1: Resistor, Resistor_THT:R_Axial_DIN0204_L3.6mm_D1.6mm_P5.08mm_Horizontal, symbol ScottoKeebs:Placeholder_Resistor
Connections:
- new net: D44.2 (DOUT), D45.4 (DIN)
- new net: D43.2 (DOUT), D44.4 (DIN)
- new net: D59.2 (DOUT), D60.4 (DIN)
- new net: D58.2 (DOUT), D59.4 (DIN)
- new net: D61.2 (DOUT), D62.4 (DIN)
- new net: D60.2 (DOUT), D61.4 (DIN)
- new net: D24.2 (DOUT), D25.4 (DIN)
- new net: D23.2 (DOUT), D24.4 (DIN)
- new net: D22.2 (DOUT), D23.4 (DIN)
- new net: D28.2 (DOUT), D29.4 (DIN)
- new net: D27.2 (DOUT), D28.4 (DIN)
- new net: D19.2 (DOUT), D20.4 (DIN)
- new net: D18.2 (DOUT), D19.4 (DIN)
- new net: D21.2 (DOUT), D22.4 (DIN)
- new net: D20.2 (DOUT), D21.4 (DIN)
- new net: D25.2 (DOUT), D26.4 (DIN)
- new net: D39.2 (DOUT), D40.4 (DIN)
- new net: D38.2 (DOUT), D39.4 (DIN)
- new net: D63.2 (DOUT), D64.4 (DIN)
- new net: D8.2 (DOUT), D9.4 (DIN)
- new net: D7.2 (DOUT), D8.4 (DIN)
- new net: D3.2 (DOUT), D4.4 (DIN)
- new net: D2.2 (DOUT), D3.4 (DIN)
- new net: D11.2 (DOUT), D12.4 (DIN)
- new net: D10.2 (DOUT), D11.4 (DIN)
- new net: D4.2 (DOUT), D5.4 (DIN)
- new net: D45.2 (DOUT), D46.4 (DIN)
- new net: D57.2 (DOUT), D58.4 (DIN)
- new net: D56.2 (DOUT), D57.4 (DIN)
- new net: D14.2 (DOUT), D15.4 (DIN)
- new net: D13.2 (DOUT), D14.4 (DIN)
- new net: D41.2 (DOUT), D42.4 (DIN)
- new net: D40.2 (DOUT), D41.4 (DIN)
- new net: D62.2 (DOUT), D63.4 (DIN)
- new net: D10.4 (DIN), D9.2 (DOUT)
- new net: D54.2 (DOUT), D55.4 (DIN)
- new net: D53.2 (DOUT), D54.4 (DIN)
- new net: D17.2 (DOUT), D18.4 (DIN)
- new net: D16.2 (DOUT), D17.4 (DIN)
- new net: D47.2 (DOUT), D48.4 (DIN)
- new net: D46.2 (DOUT), D47.4 (DIN)
- new net: D52.2 (DOUT), D53.4 (DIN)
- new net: D51.2 (DOUT), D52.4 (DIN)
- new net: D37.2 (DOUT), D38.4 (DIN)
- new net: D36.2 (DOUT), D37.4 (DIN)
- new net: D35.2 (DOUT), D36.4 (DIN)
- new net: D31.2 (DOUT), D32.4 (DIN)
- new net: D30.2 (DOUT), D31.4 (DIN)
- new net: D49.2 (DOUT), D50.4 (DIN)
- new net: D48.2 (DOUT), D49.4 (DIN)
- new net: D12.2 (DOUT), D13.4 (DIN)
- new net: D6.2 (DOUT), D7.4 (DIN)
- new net: D5.2 (DOUT), D6.4 (DIN)
- new net: D1.2 (DOUT), D2.4 (DIN)
- new net: D1.4 (DIN), R1.2
- new net: D26.2 (DOUT), D27.4 (DIN)
- new net: D15.2 (DOUT), D16.4 (DIN)
- new net: D29.2 (DOUT), D30.4 (DIN)
- new net: D34.2 (DOUT), D35.4 (DIN)
- new net: D55.2 (DOUT), D56.4 (DIN)
- new net: D50.2 (DOUT), D51.4 (DIN)
- new net: D32.2 (DOUT), D33.4 (DIN)
- new net: D33.2 (DOUT), D34.4 (DIN)
- new net: D42.2 (DOUT), D43.4 (DIN)
- new net 5v: D1.1 (VDD), D10.1 (VDD), D11.1 (VDD), D12.1 (VDD), D13.1 (VDD), D14.1 (VDD), D15.1 (VDD), D16.1 (VDD), D17.1 (VDD), D18.1 (VDD), D19.1 (VDD), D2.1 (VDD), D20.1 (VDD), D21.1 (VDD), D22.1 (VDD), D23.1 (VDD), D24.1 (VDD), D25.1 (VDD), D26.1 (VDD), D27.1 (VDD), D28.1 (VDD), D29.1 (VDD), D3.1 (VDD), D30.1 (VDD), D31.1 (VDD), D32.1 (VDD), D33.1 (VDD), D34.1 (VDD), D35.1 (VDD), D36.1 (VDD), D37.1 (VDD), D38.1 (VDD), D39.1 (VDD), D4.1 (VDD), D40.1 (VDD), D41.1 (VDD), D42.1 (VDD), D43.1 (VDD), D44.1 (VDD), D45.1 (VDD), D46.1 (VDD), D47.1 (VDD), D48.1 (VDD), D49.1 (VDD), D5.1 (VDD), D50.1 (VDD), D51.1 (VDD), D52.1 (VDD), D53.1 (VDD), D54.1 (VDD), D55.1 (VDD), D56.1 (VDD), D57.1 (VDD), D58.1 (VDD), D59.1 (VDD), D6.1 (VDD), D60.1 (VDD), D61.1 (VDD), D62.1 (VDD), D63.1 (VDD), D64.1 (VDD), D7.1 (VDD), D8.1 (VDD), D9.1 (VDD), J1.3 (Pin_3)
- new net GND: D1.3 (VSS), D10.3 (VSS), D11.3 (VSS), D12.3 (VSS), D13.3 (VSS), D14.3 (VSS), D15.3 (VSS), D16.3 (VSS), D17.3 (VSS), D18.3 (VSS), D19.3 (VSS), D2.3 (VSS), D20.3 (VSS), D21.3 (VSS), D22.3 (VSS), D23.3 (VSS), D24.3 (VSS), D25.3 (VSS), D26.3 (VSS), D27.3 (VSS), D28.3 (VSS), D29.3 (VSS), D3.3 (VSS), D30.3 (VSS), D31.3 (VSS), D32.3 (VSS), D33.3 (VSS), D34.3 (VSS), D35.3 (VSS), D36.3 (VSS), D37.3 (VSS), D38.3 (VSS), D39.3 (VSS), D4.3 (VSS), D40.3 (VSS), D41.3 (VSS), D42.3 (VSS), D43.3 (VSS), D44.3 (VSS), D45.3 (VSS), D46.3 (VSS), D47.3 (VSS), D48.3 (VSS), D49.3 (VSS), D5.3 (VSS), D50.3 (VSS), D51.3 (VSS), D52.3 (VSS), D53.3 (VSS), D54.3 (VSS), D55.3 (VSS), D56.3 (VSS), D57.3 (VSS), D58.3 (VSS), D59.3 (VSS), D6.3 (VSS), D60.3 (VSS), D61.3 (VSS), D62.3 (VSS), D63.3 (VSS), D64.3 (VSS), D7.3 (VSS), D8.3 (VSS), D9.3 (VSS), J1.4 (Pin_4)
- new net data in: J1.2 (Pin_2), R1.1
- new net data out: D64.2 (DOUT), J1.1 (Pin_1)
